File: KiCad/SYS_StepAtten/SYS_StepAtten.kicad_pcb (KiCad board)
At the start: 2 copper layers, 122 x 84 mm, 145 parts, among them J1 RCA-Out, J10 A/D GND Jumper, J11 ADJ_L, J12 ADJ_R, J2 RCA-1, J3 RCA-2, J4 AUX-1-2, J5 Barrel_Jack 9Vdc, J6 POT_EXT Conn, J7 cfg jumper, J8 ARM SWD, J9 A/D GND Jumper, K1 TQ2SA, K10 TQ2SA, K11 TQ2SA, K12 TQ2SA, K13 TQ2SA, K14 TQ2SA, K2 TQ2SA, K3 TQ2SA, K4 TQ2SA, K5 TQ2SA, K6 TQ2SA, K7 TQ2SA, K8 TQ2SA, K9 TQ2SA, Q1 2N7002, Q10 2N7002, Q11 2N7002, Q12 2N7002, Q13 2N7002, Q14 2N7002, Q2 2N7002, Q3 2N7002, Q4 2N7002, Q5 2N7002, Q6 2N7002, Q7 2N7002, Q8 2N7002, Q9 2N7002, SW1 INPUT_SWITCH, SW2 ON/OFF, U1 LM317, U2 MC34063AD, U4 STM32f030K6T6

Commit message: add uncommitted changes
Parts:
- removed D11, D12: 1N4001, Diode_SMD:D_SOD-123F
- removed G1: BarrelPolarity_CenterPos, BarrelPolarity_3mm:BarrelPolarity_3mm_CenterPos
- removed J5: Barrel_Jack 9Vdc, Connector_BarrelJack:BarrelJack_Horizontal
- removed K10, K11, K12, K13, K14, K7, K8, K9: TQ2SA, Panasonic_TQ2SA:Panasonic_TQ2SA
- removed Q1, Q2, Q3: 2N7002, Package_TO_SOT_SMD:SOT-23
- added C12: 1uf, Capacitor_SMD:C_0603_1608Metric, F.Cu at (237.3, 154.3)
- added C17: 20pF, Capacitor_SMD:C_0402_1005Metric, F.Cu at (259.7, 144.0)
- added C18: 20pF, Capacitor_SMD:C_0402_1005Metric, F.Cu at (259.7, 145.9)
- added C3: 0u1, Capacitor_SMD:C_0603_1608Metric, F.Cu at (252.2, 140.3)
- added D1: LED, LED_SMD:LED_0603_1608Metric, F.Cu at (256.3, 140.3)
- added D2: LED, LED_SMD:LED_0603_1608Metric, F.Cu at (256.3, 142.9)
- added D8: LED, LED_SMD:LED_0603_1608Metric, F.Cu at (256.3, 148.1)
- added J13: USB_C_Receptacle_USB2.0_16P, GCT_USB4210:GCT_USB4210-GF-A_REVA, F.Cu at (218.1, 149.5)
- added K15: IM03, Relay_SMD:Relay_2P2T_10x6mm_TE_IMxxG, F.Cu at (209.9, 87.3)
- added K16: IM03, Relay_SMD:Relay_2P2T_10x6mm_TE_IMxxG, F.Cu at (257.9, 121.7)
- added K17: IM03, Relay_SMD:Relay_2P2T_10x6mm_TE_IMxxG, F.Cu at (219.7, 133.2)
- added K18: IM03, Relay_SMD:Relay_2P2T_10x6mm_TE_IMxxG, F.Cu at (229.2, 133.2)
- added K19: IM03, Relay_SMD:Relay_2P2T_10x6mm_TE_IMxxG, F.Cu at (238.8, 133.2)
- added L1: MH2029-300Y, Inductor_SMD:L_0805_2012Metric, F.Cu at (256.5, 150.7)
- added R17: 500R, Resistor_SMD:R_0603_1608Metric, F.Cu at (252.2, 150.3)
- added R4: 500R, Resistor_SMD:R_0603_1608Metric, F.Cu at (252.2, 142.8)
- added R5: 500R, Resistor_SMD:R_0603_1608Metric, F.Cu at (252.2, 145.3)
- added R54: 10K, Resistor_SMD:R_0603_1608Metric, F.Cu at (252.2, 152.8)
- added R6: 500R, Resistor_SMD:R_0603_1608Metric, F.Cu at (252.2, 147.8)
- added R63: 5K1, Resistor_SMD:R_0603_1608Metric, F.Cu at (237.3, 156.8)
- added R64: 5K1, Resistor_SMD:R_0603_1608Metric, F.Cu at (237.3, 159.4)
- added R65: 22R, Resistor_SMD:R_0402_1005Metric, F.Cu at (259.7, 140.0)
- added R66: 22R, Resistor_SMD:R_0402_1005Metric, F.Cu at (259.7, 142.0)
- added U3: ATmega32U4-A, Package_QFP:TQFP-44_10x10mm_P0.8mm, F.Cu at (230.4, 146.2)
- added Y1: ABM8-16.000MHZ-10-R60-B1U-T, Crystal:Crystal_SMD_Abracon_ABM8G-4Pin_3.2x2.5mm, F.Cu at (242.0, 155.4)
- D5: value 1N4001 -> LED; footprint Diode_SMD:D_SOD-123F -> LED_SMD:LED_0603_1608Metric
- K1, K2, K3, K4, K5, K6: value TQ2SA -> IM03; footprint Panasonic_TQ2SA:Panasonic_TQ2SA -> Relay_SMD:Relay_2P2T_10x6mm_TE_IMxxG
- moved D5 115.5 mm to (256.3, 145.5)
- moved K5 86.4 mm to (238.8, 121.7), turned to 0 degrees
- moved K6 64.1 mm to (248.3, 121.7), turned to 0 degrees
- moved K4 61.7 mm to (229.2, 121.7), turned to 0 degrees
- moved K1 57.6 mm to (209.6, 102.6), turned to 0 degrees
- moved K2 51.1 mm to (219.1, 102.6), turned to 0 degrees
- moved K3 50.0 mm to (219.7, 121.7), turned to 0 degrees
Connections:
- C13 pad 1: +3V3 -> +5V
- C14 pad 1: +3V3 -> +5V
- C15 pad 1: +3V3 -> +5V
- C16 pad 1: +3V3 -> +5V
- C3 pad 1: Net-(C3-Pad1) -> Net-(U2-Vin)
- C4 pad 1: Net-(C3-Pad1) -> Net-(U2-Vin)
- D13 pad 2: Net-(D13-Pad2) -> Net-(D13-A)
- D14 pad 2: Net-(D14-Pad2) -> Net-(D14-A)
- D15 pad 2: Net-(D15-Pad2) -> Net-(D15-A)
- D16 pad 2: Net-(D16-Pad2) -> Net-(D16-A)
- D17 pad 2: Net-(D17-Pad2) -> Net-(D17-A)
- D18 pad 2: Net-(D18-Pad2) -> Net-(D18-A)
- D19 pad 2: Net-(D19-Pad2) -> Net-(D19-A)
- D5 pad 1: +5V -> Net-(D5-K)
- D5 pad 2: Net-(D5-Pad2) -> Net-(D5-A)
- F1 pad 1: Net-(C3-Pad1) -> +5V
- F2 pad 2: +3V3 -> +5V
- J1 pad 1: /AGND_L -> GNDA
- J1 pad 3: /AGND_R -> GNDA
- J10 pad 5: (no net) -> unconnected-(J10-Pin_5-Pad5)
- J10 pad 6: (no net) -> unconnected-(J10-Pin_6-Pad6)
- J2 pad 1: /RCA1_GNDL -> GNDA
- J2 pad 3: /RCA1_GNDR -> GNDA
- J3 pad 1: /RCA2_GNDL -> GNDA
- J3 pad 3: /RCA2_GNDR -> GNDA
- J4 pad B_S: /AUX2_GND -> GNDA
- J4 pad T_S: /AUX1_GND -> GNDA
- J7 pad 1: +3V3 -> +5V
- J7 pad 2: +3V3 -> +5V
- J8 pad 6: (no net) -> unconnected-(J8-Pin_6-Pad6)
- J8 pad 7: (no net) -> unconnected-(J8-Pin_7-Pad7)
- J8 pad 8: (no net) -> unconnected-(J8-Pin_8-Pad8)
- J8 pad 9: (no net) -> unconnected-(J8-Pin_9-Pad9)
- J9 pad 5: (no net) -> unconnected-(J9-Pin_5-Pad5)
- J9 pad 6: (no net) -> unconnected-(J9-Pin_6-Pad6)
- K1 pad 2: (no net) -> /AUX1_R
- K1 pad 3: (no net) -> /AUX_R
- K1 pad 4: (no net) -> /AUX2_R
- K1 pad 5: (no net) -> /AUX2_L
- K1 pad 6: (no net) -> /AUX_L
- K1 pad 7: /AUX2_GND -> /AUX1_L
- K1 pad 8: Net-(K1-Pad8) -> Net-(D14-A)
- K2 pad 2: /RCA1_GNDR -> /RCA_R
- K2 pad 3: Net-(K2-Pad3) -> /R
- K2 pad 4: /RCA2_GNDR -> /AUX_R
- K2 pad 5: (no net) -> /AUX_L
- K2 pad 6: (no net) -> /L
- K2 pad 7: /RCA2_GNDL -> /RCA_L
- K2 pad 8: Net-(K2-Pad8) -> Net-(D15-A)
- K3 pad 2: Net-(K2-Pad3) -> Net-(K3-Pad2)
- K3 pad 3: /AGND_R -> Net-(K3-Pad3)
- K3 pad 4: Net-(K1-Pad8) -> /R
- K3 pad 5: (no net) -> /L
- K3 pad 6: (no net) -> Net-(K3-Pad6)
- K3 pad 7: Net-(K1-Pad8) -> Net-(K3-Pad7)
- K3 pad 8: /AGND_L -> Net-(D16-A)
- K4 pad 2: /RCA1_R -> Net-(K4-Pad2)
- K4 pad 4: /RCA2_R -> Net-(K3-Pad3)
- K4 pad 5: (no net) -> Net-(K3-Pad6)
- K4 pad 6: (no net) -> Net-(K4-Pad6)
- K4 pad 7: /RCA2_L -> Net-(K4-Pad7)
- K4 pad 8: Net-(K4-Pad8) -> Net-(D17-A)
- K5 pad 2: /AUX1_R -> Net-(K5-Pad2)
- K5 pad 4: /AUX2_R -> Net-(K4-Pad3)
- K5 pad 5: (no net) -> Net-(K4-Pad6)
- K5 pad 6: (no net) -> Net-(K5-Pad6)
- K5 pad 7: /AUX2_L -> Net-(K5-Pad7)
- K5 pad 8: Net-(K5-Pad8) -> Net-(D18-A)
- K6 pad 2: Net-(K4-Pad3) -> Net-(K6-Pad2)
- K6 pad 3: Net-(K6-Pad3) -> Net-(K16-Pad4)
- K6 pad 5: (no net) -> Net-(K5-Pad6)
- K6 pad 6: (no net) -> Net-(K16-Pad5)
- K6 pad 7: Net-(K5-Pad8) -> Net-(K6-Pad7)
- K6 pad 8: Net-(K6-Pad8) -> Net-(D19-A)
- Q10 pad 3: Net-(D19-Pad2) -> Net-(D19-A)
- Q4 pad 1: /rly_selectL_2 -> /rly_selectL_3
- Q4 pad 3: Net-(D13-Pad2) -> Net-(D13-A)
- Q5 pad 3: Net-(D14-Pad2) -> Net-(D14-A)
- Q6 pad 3: Net-(D15-Pad2) -> Net-(D15-A)
- Q7 pad 3: Net-(D16-Pad2) -> Net-(D16-A)
- Q8 pad 3: Net-(D17-Pad2) -> Net-(D17-A)
- Q9 pad 3: Net-(D18-Pad2) -> Net-(D18-A)
- R1 pad 1: +3V3 -> +5V
- R10 pad 1: /AGND_R -> GNDA
- R10 pad 2: Net-(K7-Pad2) -> Net-(K3-Pad2)
- R11 pad 1: Net-(K7-Pad8) -> Net-(K3-Pad6)
- R11 pad 2: Net-(K6-Pad8) -> /L
- R12 pad 1: Net-(K7-Pad3) -> Net-(K3-Pad3)
- R12 pad 2: Net-(K6-Pad3) -> /R
- R13 pad 1: /AGND_L -> GNDA
- R13 pad 2: Net-(K8-Pad9) -> Net-(K4-Pad7)
- R14 pad 1: /AGND_R -> GNDA
- R14 pad 2: Net-(K8-Pad2) -> Net-(K4-Pad2)
- R15 pad 1: Net-(K8-Pad8) -> Net-(K4-Pad6)
- R15 pad 2: Net-(K7-Pad8) -> Net-(K3-Pad6)
- R16 pad 1: Net-(K8-Pad3) -> Net-(K4-Pad3)
- R16 pad 2: Net-(K7-Pad3) -> Net-(K3-Pad3)
- R18 pad 1: /AGND_L -> GNDA
- R18 pad 2: Net-(K9-Pad9) -> Net-(K5-Pad7)
- R19 pad 1: /AGND_R -> GNDA
- R19 pad 2: Net-(K9-Pad2) -> Net-(K5-Pad2)
- R20 pad 1: Net-(K10-Pad7) -> Net-(K5-Pad6)
- R20 pad 2: Net-(K8-Pad8) -> Net-(K4-Pad6)
- R21 pad 1: Net-(K10-Pad4) -> Net-(K5-Pad3)
- R21 pad 2: Net-(K8-Pad3) -> Net-(K4-Pad3)
- R22 pad 1: /AGND_L -> GNDA
- R22 pad 2: Net-(K10-Pad9) -> Net-(K6-Pad7)
- R23 pad 1: /AGND_R -> GNDA
- R23 pad 2: Net-(K10-Pad2) -> Net-(K6-Pad2)
- R24 pad 1: Net-(K10-Pad8) -> Net-(K16-Pad5)
- R24 pad 2: Net-(K10-Pad7) -> Net-(K5-Pad6)
- R25 pad 1: Net-(K10-Pad3) -> Net-(K16-Pad4)
- R25 pad 2: Net-(K10-Pad4) -> Net-(K5-Pad3)
- R26 pad 1: /AGND_L -> GNDA
- R27 pad 1: /AGND_R -> GNDA
- R28 pad 2: Net-(K10-Pad8) -> Net-(K16-Pad5)
- R29 pad 2: Net-(K10-Pad3) -> Net-(K16-Pad4)
- R30 pad 1: /AGND_L -> GNDA
- R31 pad 1: /AGND_R -> GNDA
- R38 pad 1: /AGND_L -> GNDA
- R39 pad 1: /AGND_R -> GNDA
- R51 pad 2: /AGND_L -> GNDA
- R53 pad 2: /AGND_R -> GNDA
- R54 pad 2: Net-(C3-Pad1) -> Net-(U2-Vin)
- R9 pad 1: /AGND_L -> GNDA
- R9 pad 2: Net-(K7-Pad9) -> Net-(K3-Pad7)
- RV1 pad 3: +3V3 -> +5V
- SW1 pad 1: (no net) -> unconnected-(SW1A-A-Pad1)
- SW1 pad 2: (no net) -> unconnected-(SW1A-B-Pad2)
- SW1 pad 3: (no net) -> unconnected-(SW1A-C-Pad3)
- SW1 pad 6: +3V3 -> +5V
- U1 pad 3: Net-(C3-Pad1) -> unconnected-(U1-VI-Pad3)
- U2 pad 6: Net-(C3-Pad1) -> Net-(U2-Vin)
- U4 pad 1: +3V3 -> unconnected-(U4-VDD-Pad1)
- U4 pad 10: /rly_atten4 -> /rly_atten3
- U4 pad 11: /rly_atten5 -> /rly_atten4
- U4 pad 12: /rly_atten6 -> /rly_atten5
- U4 pad 13: /extctrl_sense -> /rly_atten6
- U4 pad 18: /rly_selectL_1 -> /extctrl_sense
- U4 pad 19: /rly_selectL_2 -> /rly_selectL_1
- U4 pad 2: (no net) -> unconnected-(U4-PF0-Pad2)
- U4 pad 20: (no net) -> /rly_selectL_2
- U4 pad 21: /led1 -> unconnected-(U4-PA11-Pad21)
- U4 pad 22: /rly_mute -> /led1
- U4 pad 23: /SWDIO -> /rly_mute
- U4 pad 24: /SWDCLK -> /SWDIO
- U4 pad 25: /btn -> /SWDCLK
- U4 pad 3: (no net) -> unconnected-(U4-PF1-Pad3)
- U4 pad 5: +3V3 -> unconnected-(U4-VDDA-Pad5)
- U4 pad 6: /rly_atten0 -> unconnected-(U4-PA0-Pad6)
- U4 pad 7: /rly_atten1 -> /rly_atten0
- U4 pad 8: /rly_atten2 -> /rly_atten1
- U4 pad 9: /rly_atten3 -> /rly_atten2
Routing:
- net (no net): track 0.00 -> 321.5 mm, vias 0 -> 18
- net Net-(K6-Pad3): track 207.4 -> 0.00 mm, vias 2 -> 0
- net /R: track 0.00 -> 207.4 mm, vias 0 -> 2
- net Net-(K6-Pad8): track 194.5 -> 0.00 mm, vias 2 -> 0
- net /L: track 0.00 -> 194.5 mm, vias 0 -> 2
- net GNDA: track 0.00 -> 131.3 mm, vias 0 -> 13
- net Net-(D16-Pad2): track 57.7 -> 0.00 mm, vias 2 -> 0
- net Net-(D16-A): track 0.00 -> 57.7 mm, vias 0 -> 2
- net Net-(D19-Pad2): track 47.2 -> 0.00 mm, vias 2 -> 0
- net Net-(D19-A): track 0.00 -> 47.2 mm, vias 0 -> 2
- net Net-(K1-Pad8): track 45.0 -> 0.00 mm, vias 3 -> 0
- net Net-(D18-A): track 0.00 -> 43.8 mm, vias 0 -> 2
- net Net-(D18-Pad2): track 43.8 -> 0.00 mm, vias 2 -> 0
- net /AGND_R: track 383.4 -> 340.2 mm, vias 16 -> 6
- net Net-(D17-Pad2): track 40.3 -> 0.00 mm, vias 2 -> 0
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Other:
- net class Default removed

Commit message: WIP
Parts:
- removed C10, C4, C8: 0u1, Capacitor_SMD:C_0603_1608Metric
- removed the C3 at (116.5, 87.0)
- removed C5: 1uf, Capacitor_SMD:C_0603_1608Metric
- removed C6: 47pf, Capacitor_SMD:C_0603_1608Metric
- removed C7: 470u, Capacitor_SMD:CP_Elec_8x10.5
- removed the D1 at (102.6, 96.5)
- removed D10: LED_RGBA, RGB_LED_1.6x1.6x0:RGB_LED_1.6x1.6x0.6
- removed J10, J9: A/D GND Jumper, Connector_PinHeader_2.54mm:PinHeader_2x03_P2.54mm_Vertical
- removed J8: ARM SWD, Connector_PinHeader_1.27mm:PinHeader_2x05_P1.27mm_Vertical_SMD
- removed the L1 at (98.7, 96.5)
- removed the R17 at (177.2, 116.2)
- removed the R4 at (181.0, 144.1)
- removed the R5 at (181.0, 142.2)
- removed the R54 at (117.2, 95.2)
- removed R55: 3K8, Resistor_SMD:R_0603_1608Metric
- removed R56: 1K2, Resistor_SMD:R_0603_1608Metric
- removed the R6 at (181.0, 140.3)
- removed R7: 1K, Resistor_SMD:R_0603_1608Metric
- removed R8: 1K5, Resistor_SMD:R_0603_1608Metric
- removed TP1: nrst, TestPoint:TestPoint_Pad_2.5x2.5mm
- removed TP2: debug, TestPoint:TestPoint_Pad_2.5x2.5mm
- removed U1: LM317, Package_TO_SOT_SMD:TO-252-2
- removed U2: MC34063AD, Package_SO:SOIC-8_3.9x4.9mm_P1.27mm
- removed U4: STM32f030K6T6, Package_QFP:LQFP-32_7x7mm_P0.8mm
- moved Q6 159.7 mm to (37.7, 139.3)
- moved D15 150.7 mm to (52.7, 136.1)
- moved K16 145.2 mm to (114.0, 101.5)
- moved Q4 141.8 mm to (37.7, 130.1)
- moved JP1 141.2 mm to (37.3, 121.4), turned to 0 degrees
- moved R57 139.1 mm to (57.3, 123.9), turned to 0 degrees
- moved K17 138.0 mm to (85.3, 101.6)
- moved K18 138.0 mm to (94.9, 101.6)
- moved K19 138.0 mm to (104.4, 101.6)
- moved K3 138.0 mm to (85.3, 90.0)
- moved K4 138.0 mm to (94.9, 90.0)
- moved K5 138.0 mm to (104.4, 90.0)
- moved K6 138.0 mm to (114.0, 90.0)
- moved R58 137.6 mm to (57.3, 126.4)
- moved J7 136.6 mm to (61.6, 117.1), turned to 0 degrees
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Routing:
- net +5V: track 639.7 -> 0.00 mm, vias 37 -> 0
- net GND: track 544.6 -> 0.00 mm, vias 33 -> 0
- net /AGND_R: track 340.2 -> 0.00 mm, vias 6 -> 0
- net (no net): track 321.5 -> 0.00 mm, vias 18 -> 0
- net /AGND_L: track 260.7 -> 0.00 mm, vias 5 -> 0
- net +3V3: track 209.6 -> 0.00 mm, vias 14 -> 0
- net /R: track 207.4 -> 0.00 mm, vias 2 -> 0
- net /L: track 194.5 -> 0.00 mm, vias 2 -> 0
- net Net-(J6-Pin_4): track 186.3 -> 0.00 mm, vias 3 -> 0
- net Net-(J6-Pin_2): track 172.8 -> 0.00 mm, vias 3 -> 0
- net /rly_atten6: track 153.9 -> 0.00 mm, vias 2 -> 0
- net /rly_mute: track 135.9 -> 0.00 mm, vias 2 -> 0
- net /rly_atten0: track 134.8 -> 0.00 mm, vias 2 -> 0
- net GNDA: track 131.3 -> 0.00 mm, vias 13 -> 0
- net /rly_atten5: track 124.5 -> 0.00 mm, vias 2 -> 0
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- removed copper zone on B.Cu, net +3V3
- removed copper zone on F.Cu, net /AGND_L
- removed copper zone on F.Cu, net /AGND_R
- removed copper zone on B.Cu, net GND
- removed copper zone on F.Cu, net GND

Commit message: Redo relay layout
Parts:
- removed SW2: ON/OFF, Connector_PinHeader_2.54mm:PinHeader_1x02_P2.54mm_Vertical
- added TP1: nrst, TestPoint:TestPoint_Pad_2.5x2.5mm, F.Cu at (194.9, 120.4)
- added TP2: debug, TestPoint:TestPoint_Pad_2.5x2.5mm, F.Cu at (194.9, 124.2)
- D13, D14, D15, D16, D17, D18, D19, D20, D21, D22, D23: footprint Diode_SMD:D_SOD-123F -> Diode_THT:D_DO-35_SOD27_P7.62mm_Horizontal
- moved D16 145.3 mm to (192.7, 100.6), turned to -90 degrees
- moved R10 145.1 mm to (185.7, 98.0), turned to 180 degrees
- moved R9 144.3 mm to (185.6, 110.7), turned to 180 degrees
- moved R12 141.3 mm to (181.4, 98.0), turned to 180 degrees
- moved D15 140.3 mm to (183.4, 85.1), turned to -90 degrees
- moved R11 140.1 mm to (181.3, 110.7), turned to 180 degrees
- moved R14 133.7 mm to (172.9, 98.0), turned to 180 degrees
- moved D17 132.9 mm to (178.7, 100.6), turned to -90 degrees
- moved JP1 132.2 mm to (169.2, 129.5), turned to 180 degrees
- moved R13 131.9 mm to (172.9, 110.7), turned to 180 degrees
- moved R16 130.4 mm to (168.6, 98.0), turned to 180 degrees
- moved R15 127.9 mm to (168.5, 110.7), turned to 180 degrees
- moved C1 125.8 mm to (160.8, 130.3)
- moved Q6 125.2 mm to (161.9, 123.1)
- moved D13 123.4 mm to (168.0, 85.1), turned to -90 degrees
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- renumbered K18 to K10, K19 to K11, K15 to K3, K3 to K4, K4 to K5, K5 to K6, K6 to K7, K16 to K8, K17 to K9
Connections:
- D3 pad 1: +3V3 -> +5V
- D6 pad 1: +3V3 -> +5V
- F1 pad 2: Net-(SW2-B) -> Net-(U3-VBUS)
- J13 pad A4: Net-(SW2-A) -> Net-(U3-VBUS)
- J13 pad A9: Net-(SW2-A) -> Net-(U3-VBUS)
- J13 pad B4: Net-(SW2-A) -> Net-(U3-VBUS)
- J13 pad B9: Net-(SW2-A) -> Net-(U3-VBUS)
- J13 pad SH1: (no net) -> GND
- J13 pad SH2: (no net) -> GND
- J13 pad SH3: (no net) -> GND
- J13 pad SH4: (no net) -> GND
- U3 pad 7: Net-(SW2-A) -> Net-(U3-VBUS)
Routing:
- net /AUX_R: track 0.00 -> 39.9 mm
- net /AUX_L: track 0.00 -> 35.4 mm
- net /RCA_R: track 0.00 -> 34.4 mm
- net /RCA_L: track 0.00 -> 34.3 mm
- net /RCA2_L: track 0.00 -> 27.9 mm
- net /AUX1_R: track 0.00 -> 25.8 mm
- net /RCA1_R: track 0.00 -> 25.8 mm
- net /AUX1_L: track 0.00 -> 24.2 mm
- net /RCA1_L: track 0.00 -> 20.3 mm
- net +5V: track 0.00 -> 17.8 mm
- net Net-(J11-Pin_2): track 0.00 -> 15.3 mm
- net Net-(J12-Pin_2): track 0.00 -> 14.1 mm
- net /RCA2_R: track 0.00 -> 13.5 mm
- net GND: track 0.00 -> 12.1 mm
- net /AUX2_R: track 0.00 -> 11.3 mm
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Other:
- board text added: "[https://github.com/Max585t/SYS_StepAtten]"
- board text removed: "1"
- board text removed: "2"
- board text removed: "AGnd-DGnd:"
- board text removed: "L"
- board text removed: "NO-YES"
- board text removed: "ON/OFF"
- board text removed: "R"
- board text removed: "RCA LGND-RGND"
- board text removed: "SCHILK"
- board text removed: "[https://github.com/TheSchilk/SYS_StepAtten]"
- board text removed: "v1.3"

Commit message: Sync work done on laptop
finished relay layout
Parts:
- added D9: 1N4001, Diode_SMD:D_SOD-123, B.Cu at (176.7, 88.8)
- added J5: RJ9, 615004143821:615004143821, F.Cu at (192.5, 104.9)
- added J8: Conn_02x02_Odd_Even, Connector_PinHeader_2.54mm:PinHeader_2x02_P2.54mm_Vertical, F.Cu at (194.6, 93.3)
- added J9: AudioJack3, Connector_Audio:Jack_3.5mm_CUI_SJ-3523-SMT_Horizontal, F.Cu at (127.5, 68.6)
- added K12: IME03, Relay_SMD:Relay_2P2T_10x6mm_TE_IMxxG, F.Cu at (176.7, 85.0)
- added Q1: 2N7002, Package_TO_SOT_SMD:SOT-23, F.Cu at (156.7, 102.9)
- added R7: 10K, Resistor_SMD:R_0603_1608Metric, F.Cu at (156.8, 105.8)
- added R8: 10K, Resistor_SMD:R_0603_1608Metric, F.Cu at (179.7, 120.4)
- added SW2: SW_MEC_5G, E_Switch:Untitled, F.Cu at (186.0, 140.1)
- D13, D14, D15, D16, D17, D18, D19, D20, D21, D22, D23: footprint Diode_THT:D_DO-35_SOD27_P7.62mm_Horizontal -> Diode_SMD:D_SOD-123; moved to B.Cu
- J4: value AUX-1-2 -> AudioJack3; footprint 3.5mm_RiserPCB:3.5mm_RiserPCB -> Connector_Audio:Jack_3.5mm_CUI_SJ-3523-SMT_Horizontal
- J6: footprint Connector_PinHeader_2.54mm:PinHeader_2x02_P2.54mm_Horizontal -> Connector_PinHeader_2.54mm:PinHeader_2x02_P2.54mm_Vertical
- K1, K2, K3: value IM03 -> IME03
- moved R36 100.8 mm to (144.8, 126.1), turned to 90 degrees
- moved K11 100.5 mm to (86.6, 90.8), turned to 0 degrees
- moved R37 100.3 mm to (144.8, 129.9), turned to 90 degrees
- moved Q10 99.0 mm to (142.3, 129.9), turned to 180 degrees
- moved R35 98.7 mm to (144.8, 118.6), turned to 90 degrees
- moved R40 98.0 mm to (144.8, 122.3), turned to 90 degrees
- moved Q11 97.5 mm to (142.3, 126.1), turned to 180 degrees
- moved Q9 96.6 mm to (142.3, 122.3), turned to 180 degrees
- moved R41 96.3 mm to (144.8, 114.7), turned to 90 degrees
- moved R34 96.2 mm to (144.8, 110.7), turned to 90 degrees
- moved Q12 95.4 mm to (142.3, 118.6), turned to 180 degrees
- moved Q8 94.7 mm to (142.3, 114.7), turned to 180 degrees
- moved R44 94.6 mm to (144.7, 106.9), turned to 90 degrees
- moved R47 94.4 mm to (144.7, 103.0), turned to 90 degrees
- moved Q13 93.0 mm to (142.2, 110.7), turned to 180 degrees
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Connections:
- net Net-(J13-D+-PadA6) renamed /D+
- net Net-(J13-D--PadA7) renamed /D-
- net Net-(J6-Pin_2) renamed /e_p
- net Net-(J6-Pin_4) renamed /e_s
- net Net-(U3-VBUS) renamed VBUS
- J1 pad 1: GNDA -> GND
- J1 pad 3: GNDA -> GND
- J2 pad 1: GNDA -> GND
- J2 pad 3: GNDA -> GND
- J3 pad 1: GNDA -> GND
- J3 pad 3: GNDA -> GND
- K1 pad 2: /AUX1_R -> unconnected-(K1-Pad2)
- K1 pad 3: /AUX_R -> /R
- K1 pad 4: /AUX2_R -> /AUX1_R
- K1 pad 5: /AUX2_L -> /AUX1_L
- K1 pad 6: /AUX_L -> /L
- K1 pad 7: /AUX1_L -> unconnected-(K1-Pad7)
- K11 pad 2: GNDA -> GND
- K11 pad 7: GNDA -> GND
- K2 pad 2: /RCA_R -> unconnected-(K2-Pad2)
- K2 pad 4: /AUX_R -> /AUX2_R
- K2 pad 5: /AUX_L -> /AUX2_L
- K2 pad 7: /RCA_L -> unconnected-(K2-Pad7)
- K3 pad 2: /RCA1_R -> unconnected-(K3-Pad2)
- K3 pad 3: /RCA_R -> /R
- K3 pad 6: /RCA_L -> /L
- K3 pad 7: /RCA1_L -> unconnected-(K3-Pad7)
- R10 pad 1: GNDA -> GND
- R13 pad 1: GNDA -> GND
- R14 pad 1: GNDA -> GND
- R18 pad 1: GNDA -> GND
- R19 pad 1: GNDA -> GND
- R22 pad 1: GNDA -> GND
- R23 pad 1: GNDA -> GND
- R26 pad 1: GNDA -> GND
- R27 pad 1: GNDA -> GND
- R30 pad 1: GNDA -> GND
- R31 pad 1: GNDA -> GND
- R38 pad 1: GNDA -> GND
- R39 pad 1: GNDA -> GND
- R51 pad 2: GNDA -> GND
- R53 pad 2: GNDA -> GND
- R9 pad 1: GNDA -> GND
- U3 pad 10: /rly_atten2 -> Net-(D5-A)
- U3 pad 11: /rly_atten3 -> Net-(D8-A)
- U3 pad 12: /rly_mute -> unconnected-(U3-PB7-Pad12)
- U3 pad 18: Net-(D1-A) -> unconnected-(U3-PD0-Pad18)
- U3 pad 19: Net-(D2-A) -> unconnected-(U3-PD1-Pad19)
- U3 pad 20: Net-(D5-A) -> /rly_selectL_4
- U3 pad 21: Net-(D8-A) -> /rly_selectL_3
- U3 pad 22: unconnected-(U3-PD5-Pad22) -> /rly_selectL_2
- U3 pad 25: unconnected-(U3-PD4-Pad25) -> /rly_mute
- U3 pad 26: /extctrl_sense -> /rly_atten6
- U3 pad 27: /btn -> /rly_atten0
- U3 pad 28: /rly_atten4 -> /rly_atten5
- U3 pad 29: /rly_atten5 -> /rly_atten1
- U3 pad 30: /rly_atten6 -> /rly_atten4
- U3 pad 31: /cfg2 -> /rly_atten2
- U3 pad 32: /cfg1 -> /rly_atten3
- U3 pad 33: unconnected-(U3-~{HWB}/PE2-Pad33) -> /rly_selectL_1
- U3 pad 36: unconnected-(U3-PF7-Pad36) -> /poti
- U3 pad 37: /poti -> /extctrl_sense
- U3 pad 39: /rly_selectL_3 -> /cfg1
- U3 pad 40: /rly_selectL_2 -> /cfg2
- U3 pad 41: /rly_selectL_1 -> /btn
- U3 pad 8: /rly_atten0 -> Net-(D1-A)
- U3 pad 9: /rly_atten1 -> Net-(D2-A)
Routing:
- net +5V: track 17.8 -> 439.0 mm, vias 0 -> 21
- net /D+: track 2.04 -> 160.5 mm, vias 0 -> 2
- net /D-: track 6.67 -> 164.7 mm, vias 2 -> 3
- net /L: track 0.00 -> 156.9 mm
- net /R: track 0.00 -> 143.0 mm, vias 0 -> 2
- net VBUS: track 3.50 -> 138.8 mm, vias 0 -> 4
- net GND: track 12.1 -> 89.5 mm, vias 0 -> 71
- net Net-(D1-A): track 0.00 -> 65.6 mm, vias 0 -> 2
- net Net-(D23-A): track 0.00 -> 60.5 mm, vias 0 -> 2
- net Net-(D22-A): track 0.00 -> 59.1 mm, vias 0 -> 2
- net Net-(D2-A): track 0.00 -> 58.9 mm, vias 0 -> 2
- net Net-(D21-A): track 0.00 -> 57.6 mm, vias 0 -> 2
- net Net-(D20-A): track 0.00 -> 55.7 mm, vias 0 -> 2
- net Net-(D5-A): track 0.00 -> 52.5 mm, vias 0 -> 2
- net Net-(D16-A): track 0.00 -> 50.4 mm, vias 0 -> 2
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- added copper zone on In2.Cu, net +5V
- added copper zone on B.Cu, net GND
- added copper zone on F.Cu, net GND
- added copper zone on In1.Cu, net GND
- added copper zone on In2.Cu, net GND
Other:
- copper layers 2 -> 4
- board text removed: "Ext. Pot."
